Commit message: add lidar2

File: description/lidar.xacro (robot description, xacro)
@@ -4,5 +4,22 @@
         <parent link="chassis"/>
         <child link="lidar_frame"/>
-        <origin xyz="0 0 0" rpy="0 0 0"/>
+        <origin xyz="0 0 0.1" rpy="0 0 0"/>
     </joint>
+    <link name="lidar_frame">
+        <visual>
+            <geometry>
+                <cylinder radius="0.0625" length="0.023"/>
+            </geometry>
+            <materaial name="orange"/>
+        </visual>
+        <collision>
+            <geometry>
+                <cylinder radius="0.0625" length="0.023"/>
+            </geometry>
+            <materaial name="orange"/>
+        </collision>
+        <xacro:inertial_cylinder mass="0.15" length="0.023" radius="0.0625">
+            <origin xyz="0 0 0" rpy="0 0 0"/>
+        </xacro:inertial_cylinder>
+    </link>
 </robot>
