Commit message: first_simulation

File: description/gazebo_control.xacro (robot description, xacro)
@@ -9,6 +9,6 @@
             <wheel_diameter>0.125</wheel_diameter>
             <!-- Limit -->
-            <max_wheel_torque>1000</max_wheel_torque>
-            <max_wheel_acceleration>100.0</max_wheel_acceleration>
+            <max_wheel_torque>250</max_wheel_torque>
+            <max_wheel_acceleration>20.0</max_wheel_acceleration>
             <!-- Output -->
             <odometry_frame>odem</odometry_frame>

File: description/lidar.xacro (robot description, xacro)
@@ -4,10 +4,10 @@
         <parent link="chassis"/>
         <child link="lidar_frame"/>
-        <origin xyz="0 0 0.1" rpy="0 0 0"/>
+        <origin xyz="0.032 0 0.059" rpy="0 0 0"/>
     </joint>
     <link name="lidar_frame">
         <visual>
             <geometry>
-                <cylinder radius="0.0625" length="0.023"/>
+                <cylinder radius="0.035" length="0.03"/>
             </geometry>
             <materaial name="orange"/>
@@ -15,11 +15,41 @@
         <collision>
             <geometry>
-                <cylinder radius="0.0625" length="0.023"/>
+                <cylinder radius="0.035" length="0.03"/>
             </geometry>
             <materaial name="orange"/>
         </collision>
-        <xacro:inertial_cylinder mass="0.15" length="0.023" radius="0.0625">
+        <xacro:inertial_cylinder mass="0.001" length="0.03" radius="0.035">
             <origin xyz="0 0 0" rpy="0 0 0"/>
         </xacro:inertial_cylinder>
     </link>
+    <gazebo reference="lidar_frame">
+        <material>Gazebo/Red</material>
+        <sensor name="lidar" type="ray">
+            <pose>0 0 0 0 0 0</pose>
+            <visualize>true</visualize>
+            <update_rate>10</update_rate>
+            <ray>
+                <scan>
+                    <horizontal>
+                        <sample>360</sample>
+                        <resolution>1</resolution>
+                        <min_angle>-3.14</min_angle>
+                        <max_angle>3.14</max_angle>
+                    </horizontal>
+                </scan>
+                <range>
+                    <min>0.3</min>
+                    <max>12</max>
+                    <resolution>0.01</resolution>
+                </range>
+            </ray>
+            <plugin name="lidar_controller" filename="libgazebo_ros_ray_sensor.so">
+                <ros>
+                    <argument>~/out:=scan</argument>
+                </ros>
+                <output_type>sensor_msgs/LaserScan</output_type>
+                <frame_name>lidar_frame</frame_name>
+            </plugin>
+        </sensor>
+    </gazebo>
 </robot>

File: description/robot_core.xacro (robot description, xacro)
@@ -61,5 +61,5 @@
                 <cylinder radius="0.0625" length="0.023"/>
             </geometry>
-            <materaial name="blue"/>
+            <materaial name="black"/>
         </visual>
         <collision>
@@ -67,5 +67,5 @@
                 <cylinder radius="0.0625" length="0.023"/>
             </geometry>
-            <materaial name="blue"/>
+            <materaial name="black"/>
         </collision>
         <xacro:inertial_cylinder mass="0.15" length="0.023" radius="0.0625">
@@ -88,5 +88,5 @@
                 <cylinder radius="0.0625" length="0.023"/>
             </geometry>
-            <materaial name="blue"/>
+            <materaial name="black"/>
         </visual>
         <collision>
@@ -94,5 +94,5 @@
                 <cylinder radius="0.0625" length="0.023"/>
             </geometry>
-            <materaial name="blue"/>
+            <materaial name="black"/>
         </collision>
         <xacro:inertial_cylinder mass="0.15" length="0.023" radius="0.0625">
