Commit message: add caster wheel

File: description/robot_core.xacro (robot description, xacro)
@@ -47,5 +47,4 @@
     <gazebo reference="chassis">
         <material>Gazebo/Yellow</material>
-        <mu3 value="0.001"/>
     </gazebo>
     <!-- LEFT WHEEL LINK -->
@@ -76,4 +75,52 @@
         <material>Gazebo/Blue</material>
     </gazebo>
+    <!-- LEFT CASTER WHEEL LINK -->
+    <joint name="left_caster_joint" type="continuous">
+        <parent link="base_link"/>
+        <child link="left_caster_link"/>
+        <origin xyz="-0.420 0.139 0.007" rpy="-${pi} 0 0"/>
+        <axis xyz="0 0 1"/>
+    </joint>
+    <link name="left_caster_link">
+        <materaial name="black"/>
+        <visual>
+            <origin xyz="0 0 0" rpy="-${pi} 0 0"/>
+            <geometry>
+                <mesh filename="file://$(find my_diff_drive_bot)/meshes/caster_link.stl" scale="0.001 0.001 0.001"/>
+            </geometry>
+        </visual>
+        <collision>
+            <origin xyz="0 0 0" rpy="-${pi} 0 0"/>
+            <geometry>
+                <mesh filename="file://$(find my_diff_drive_bot)/meshes/caster_link.stl" scale="0.001 0.001 0.001"/>
+            </geometry>
+            <materaial name="black"/>
+        </collision>
+        <xacro:inertial_cylinder mass="0.1" length="0.090" radius="0.03">
+            <origin xyz="0 0 0" rpy="0 0 0"/>
+        </xacro:inertial_cylinder>
+    </link>
+    <!-- LEFT CASTER WHEEL -->
+    <joint name="left_caster_wheel_joint" type="continuous">
+        <parent link="left_caster_link"/>
+        <child link="left_caster_wheel"/>
+        <origin xyz="0.02 0 0.04" rpy="-${pi/2} 0 0"/>
+        <axis xyz="0 0 1"/>
+    </joint>
+    <link name="left_caster_wheel">
+        <visual>
+            <geometry>
+                <cylinder radius="0.025" length="0.018"/>
+            </geometry>
+        </visual>
+        <collision>
+            <geometry>
+                <cylinder radius="0.025" length="0.018"/>
+            </geometry>
+        </collision>
+        <xacro:inertial_cylinder mass="0.1" length="0.018" radius="0.025">
+            <origin xyz="0 0 0" rpy="0 0 0"/>
+        </xacro:inertial_cylinder>
+    </link>
     <!-- RIGHT WHEEL LINK -->
     <joint name="right_wheel_joint" type="continuous">
@@ -100,6 +147,51 @@
         </xacro:inertial_cylinder>
     </link>
-    <gazebo reference="right_wheel">
-        <material>Gazebo/Blue</material>
-    </gazebo>
+      <!-- RIGHT CASTER WHEEL LINK -->
+      <joint name="right_caster_joint" type="continuous">
+        <parent link="base_link"/>
+        <child link="right_caster_link"/>
+        <origin xyz="-0.420 -0.139 0.007" rpy="-${pi} 0 0"/>
+        <axis xyz="0 0 1"/>
+    </joint>
+    <link name="right_caster_link">
+        <materaial name="black"/>
+        <visual>
+            <origin xyz="0 0 0" rpy="-${pi} 0 0"/>
+            <geometry>
+                <mesh filename="file://$(find my_diff_drive_bot)/meshes/caster_link.stl" scale="0.001 0.001 0.001"/>
+            </geometry>
+        </visual>
+        <collision>
+            <origin xyz="0 0 0" rpy="-${pi} 0 0"/>
+            <geometry>
+                <mesh filename="file://$(find my_diff_drive_bot)/meshes/caster_link.stl" scale="0.001 0.001 0.001"/>
+            </geometry>
+            <materaial name="black"/>
+        </collision>
+        <xacro:inertial_cylinder mass="0.1" length="0.090" radius="0.03">
+            <origin xyz="0 0 0" rpy="0 0 0"/>
+        </xacro:inertial_cylinder>
+    </link>
+    <!-- RIGHT CASTER WHEEL -->
+    <joint name="right_caster_wheel_joint" type="continuous">
+        <parent link="right_caster_link"/>
+        <child link="right_caster_wheel"/>
+        <origin xyz="0.02 0 0.04" rpy="-${pi/2} 0 0"/>
+        <axis xyz="0 0 1"/>
+    </joint>
+    <link name="right_caster_wheel">
+        <visual>
+            <geometry>
+                <cylinder radius="0.025" length="0.018"/>
+            </geometry>
+        </visual>
+        <collision>
+            <geometry>
+                <cylinder radius="0.025" length="0.018"/>
+            </geometry>
+        </collision>
+        <xacro:inertial_cylinder mass="0.1" length="0.018" radius="0.025">
+            <origin xyz="0 0 0" rpy="0 0 0"/>
+        </xacro:inertial_cylinder>
+    </link>
 </robot>
