Commit message: add real robot packge

File: description/robot.urdf.xacro (robot description, xacro)
@@ -1,7 +1,12 @@
 <?xml version="1.0"?>
 <robot xmlns:xacro="http://www.ros.org/wiki/xacro"  name="robot">
+    <xacro:arg name="use_ros2_contorl" default="true"/>
     <xacro:include filename="robot_core.xacro"/>
-    <!-- <xacro:include filename="gazebo_control.xacro"/> -->
-    <xacro:include filename="ros2_control.xacro"/>
+    <xacro:if value="$(arg use_ros2_contorl)">
+        <xacro:include filename="ros2_control.xacro"/>
+    </xacro:if>
+    <xacro:unless value="$(arg use_ros2_contorl)">
+        <xacro:include filename="gazebo_control.xacro"/>
+    </xacro:unless>
     <xacro:include filename="lidar.xacro"/>
 </robot>

File: description/ros2_control.xacro (robot description, xacro)
@@ -1,4 +1,30 @@
 <?xml version="1.0"?>
 <robot xmlns:xacro="http://www.ros.org/wiki/xacro">
+  <ros2_control name="RealRob0t" type="system">
+    <hardware>
+        <plugin>gazebo_ros2_control/GazeboSystem</plugin>
+    </hardware>
+    <joint name="left_wheel_joint">
+        <command_interface name="velocity">
+            <param name="min">10</param>
+            <param name="max">10</param>
+        </command_interface>
+        <state_interface name="velocity"/>
+        <state_interface name="position"/>
+    </joint>
+    <joint name="right_wheel_joint">
+        <command_interface name="velocity">
+            <param name="min">10</param>
+            <param name="max">10</param>
+        </command_interface>
+        <state_interface name="velocity"/>
+        <state_interface name="position"/>
+    </joint>
+  </ros2_control>
+  <gazebo>
+    <plugin name="gazebo_ros2_control" filename="libgazebo_ros2_control.so">
+        <parameters>$(find my_diff_drive_bot)/config/my_controllers.yaml</parameters>
+    </plugin>
+  </gazebo>
   <ros2_control name="GazeboSystem" type="system">
     <hardware>
